File: pertec_arduino_adapter/pertec_arduino_adapter.kicad_sch (KiCad schematic)
At the start: 19 parts, among them J1 Conn_02x25_Odd_Even, J2 Conn_02x25_Odd_Even, J3 POWER, J4 ANALOGL, J5 ANALOGH, J6 Conn_02x18_Odd_Even, J7 IOH, J8 IOL, J9 UART, U1 SN74AVC8T245PW, U2 SN74AVC8T245PW, U3 SN74AVC8T245PW, U4 SN74AVC8T245PW, U5 SN74AVC8T245PW, U6 SN74AVC8T245PW

Commit message: Development checkpoint: schematic complete, passes ERC, started layout.
Parts:
- removed J3: POWER, pertec_arduino_adapter:PinHeader_1x08_P2.54mm_Vertical, symbol pertec_arduino_adapter:Conn_01x08
- removed J4: ANALOGL, pertec_arduino_adapter:PinHeader_1x08_P2.54mm_Vertical, symbol pertec_arduino_adapter:Conn_01x08
- removed J5: ANALOGH, pertec_arduino_adapter:PinHeader_1x08_P2.54mm_Vertical, symbol pertec_arduino_adapter:Conn_01x08
- removed J6: Conn_02x18_Odd_Even, pertec_arduino_adapter:PinHeader_2x18_P2.54mm_Vertical_Mirror, symbol pertec_arduino_adapter:Conn_02x18_Odd_Even
- removed J7: IOH, pertec_arduino_adapter:PinHeader_1x10_P2.54mm_Vertical, symbol pertec_arduino_adapter:Conn_01x10
- removed J8: IOL, pertec_arduino_adapter:PinHeader_1x08_P2.54mm_Vertical, symbol pertec_arduino_adapter:Conn_01x08
- removed J9: UART, pertec_arduino_adapter:PinHeader_1x08_P2.54mm_Vertical, symbol pertec_arduino_adapter:Conn_01x08
- removed U1, U2, U3, U4, U5, U6: SN74AVC8T245PW, pertec_arduino_adapter:SOIC-24W_7.5x15.4mm_P1.27mm, symbol pertec_arduino_adapter:SN74AVC8T245PW
- added BT1: CR2032, pertec_arduino_adapter:BatteryHolder_Keystone_1058_1x2032, symbol pertec_arduino_adapter:Battery_Cell
- added C1, C3: (no value), symbol pertec_arduino_adapter:C_Small
- added C10, C11, C12, C13, C14, C2, C4, C5, C6, C7, C8, C9: 0.1 μF, symbol pertec_arduino_adapter:C_Small
- added J3: Conn_02x03_Odd_Even, pertec_arduino_adapter:PinSocket_2x03_P2.00mm_Vertical_Mirror, symbol pertec_arduino_adapter:Conn_02x03_Odd_Even
- added J4, J5: Conn_01x24, pertec_arduino_adapter:PinSocket_1x24_P2.54mm_Vertical, symbol pertec_arduino_adapter:Conn_01x24
- added J6: Conn_01x05, pertec_arduino_adapter:PinSocket_1x05_P2.54mm_Vertical, symbol pertec_arduino_adapter:Conn_01x05
- added J7: (no value), symbol pertec_arduino_adapter:RJ45_Cetus_J1B1211CCD
- added J8: (no value), symbol pertec_arduino_adapter:Conn_02x03_Odd_Even
- added Q1, Q2: BSS138, symbol pertec_arduino_adapter:BSS138
- added R1, R10, R11, R2, R3, R4, R5, R6, R7, R8, R9: 10 kΩ, symbol pertec_arduino_adapter:R
- added U1, U2, U3, U4, U5, U6: (no value), symbol pertec_arduino_adapter:SN74LVC8T245NSR
- added U7: PCA9535DBR, pertec_arduino_adapter:SOIC-24W_7.5x15.4mm_P1.27mm, symbol pertec_arduino_adapter:PCA9535DBR
- RN1, RN2, RN3: value (none) -> R1=220Ω, R2=330Ω; footprint (none) -> pertec_arduino_adapter:R_Array_SIP10
- RN4: value (none) -> R1=220Ω, R2=330Ω; footprint (none) -> pertec_arduino_adapter:R_Array_SIP6
Connections:
- net +3V3: now also C11.1, C13.1, C3.1, C5.1, C7.1, C9.1, J4.3 (Pin_3), J5.15 (Pin_15), Q1.1 (G), Q2.1 (G), R1.1, R10.1, R11.1, R2.1, R7.1, R9.1, U1.1 (VCCA), U2.1 (VCCA), U3.1 (VCCA), U4.1 (VCCA), U5.1 (VCCA), U6.1 (VCCA)
- net +5V: now also C10.1, C12.1, C14.1, C2.1, C4.1, C6.1, C8.1, J4.1 (Pin_1), R3.1, R4.1, U1.23 (VCCB), U1.24 (VCCB), U2.23 (VCCB), U2.24 (VCCB), U3.23 (VCCB), U3.24 (VCCB), U4.23 (VCCB), U4.24 (VCCB), U5.23 (VCCB), U5.24 (VCCB), U6.23 (VCCB), U6.24 (VCCB), U7.24 (VCC)
- net GNDREF: now also BT1.2 (-), C10.2, C11.2, C12.2, C13.2, C14.2, C2.2, C3.2, C4.2, C5.2, C6.2, C7.2, C8.2, C9.2, J4.15 (Pin_15), J4.2 (Pin_2), J5.1 (Pin_1), J6.3 (Pin_3), J8.1 (Pin_1), J8.3 (Pin_3), J8.5 (Pin_5), R5.2, R6.2, R8.2, U1.11 (GND), U1.12 (GND), U1.13 (GND), U1.2 (DIR), U1.22 (~{OE}), U2.11 (GND), U2.12 (GND), U2.13 (GND), U2.22 (~{OE}), U3.11 (GND), U3.12 (GND), U3.13 (GND), U3.2 (DIR), U3.22 (~{OE}), U4.11 (GND), U4.12 (GND), U4.13 (GND), U4.22 (~{OE}), U5.11 (GND), U5.12 (GND), U5.13 (GND), U5.2 (DIR), U5.22 (~{OE}), U6.11 (GND), U6.12 (GND), U6.13 (GND), U6.22 (~{OE}), U7.12 (GND)
- net ICER: now also U5.21 (B1)
- net IDBY: now also U3.14 (B8)
- net IDENT: now also U7.4 (P00)
- net IEDIT: now also U4.15 (B7)
- net IEOT: now also U3.19 (B3)
- net IERASE: now also U4.14 (B8)
- net IFAD: now also U7.11 (P07)
- net IFBY: now also U5.20 (B2)
- net IFEN: now also U7.9 (P05)
- net IFMK: now also U3.21 (B1)
- net IFPT: now also U3.17 (B5)
- net IGO: now also U2.19 (B3)
- net IHER: now also U1.14 (B8)
- net ILDP: now also U1.18 (B4)
- net ILOL: now also U7.15 (P12)
- net ILWD: now also U2.21 (B1)
- net INRZ: now also U7.7 (P03)
- net IOFL: now also U6.14 (B8)
- net IONL: now also U7.18 (P15)
- net IR0: now also U1.20 (B2)
- net IR1: now also U1.19 (B3)
- net IR2: now also U5.19 (B3)
- net IR3: now also U5.18 (B4)
- net IR4: now also U1.17 (B5)
- net IR5: now also U3.20 (B2)
- net IR6: now also U1.15 (B7)
- net IR7: now also U1.16 (B6)
- net IRDY: now also U3.18 (B4)
- net IREV: now also U2.16 (B6)
- net IREW: now also U2.15 (B7)
- net IRP: now also U1.21 (B1)
- net IRSTR: now also U3.16 (B6)
- net IRTH1: now also U7.17 (P14)
- net IRTH2: now also U7.16 (P13)
- net IRWD: now also U7.5 (P01)
- net ISGL: now also U7.14 (P11)
- net ISPEED: now also U7.6 (P02)
- net ITAD0: now also U7.8 (P04)
- net ITAD1: now also U7.10 (P06)
- net IW0: now also U2.18 (B4)
- net IW1: now also U2.17 (B5)
- net IW2: now also U4.18 (B4)
- net IW3: now also U4.20 (B2)
- net IW4: now also U2.20 (B2)
- net IW5: now also U4.17 (B5)
- net IW6: now also U4.19 (B3)
- net IW7: now also U4.21 (B1)
- net IWFM: now also U6.15 (B7)
- net IWP: now also U2.14 (B8)
- net IWRT: now also U4.16 (B6)
- net IWSTR: now also U3.15 (B7)
- net IHISP renamed IDEN
- net IDEN: now also U7.13 (P10)
- new net: R10.2, U4.2 (DIR)
- new net: BT1.1 (+), J6.5 (Pin_5)
- new net: R6.1, U7.2 (A1)
- new net: R8.1, U7.21 (A0)
- new net: Q2.3 (D), R4.2, U7.22 (SCL)
- new net: Q1.3 (D), R3.2, U7.23 (SDA)
- new net: R5.1, U7.3 (A2)
- new net: C1.1, J7.2 (TXC), J7.5 (RXC)
- new net: R9.2, U2.2 (DIR)
- new net: R11.2, U6.2 (DIR)
- new net ETHERNET_G: C1.2, J3.4 (Pin_4), J7.13 (SHIELD), J7.8 (GND), J7.9 (LEDG_K)
- new net ETHERNET_LED: J3.3 (Pin_3), J7.10 (LEDG_A)
- new net ETHERNET_RM: J3.6 (Pin_6), J7.6 (RX-)
- new net ETHERNET_RP: J3.5 (Pin_5), J7.4 (RX+)
- new net ETHERNET_TM: J3.1 (Pin_1), J7.3 (TX-)
- new net ETHERNET_TP: J3.2 (Pin_2), J7.1 (TX+)
- new net GPIO_AD_B0_02: J5.3 (Pin_3), U1.3 (A1)
- new net GPIO_AD_B0_03: J5.2 (Pin_2), U3.3 (A1)
- new net GPIO_AD_B0_12: J5.16 (Pin_16), Q2.2 (S), R2.2
- new net GPIO_AD_B0_13: J5.17 (Pin_17), Q1.2 (S), R1.2
- new net GPIO_AD_B1_00: J4.8 (Pin_8), U1.8 (A6)
- new net GPIO_AD_B1_01: J4.9 (Pin_9), U1.9 (A7)
- new net GPIO_AD_B1_02: J4.13 (Pin_13), U3.4 (A2)
- new net GPIO_AD_B1_03: J4.12 (Pin_12), U1.7 (A5)
- new net GPIO_AD_B1_04: J4.17 (Pin_17), U5.6 (A4)
- new net GPIO_AD_B1_05: J4.16 (Pin_16), U5.5 (A3)
- new net GPIO_AD_B1_06: J4.10 (Pin_10), U1.5 (A3)
- new net GPIO_AD_B1_07: J4.11 (Pin_11), U1.4 (A2)
- new net GPIO_AD_B1_08: J4.5 (Pin_5), U4.3 (A1)
- new net GPIO_AD_B1_09: J4.4 (Pin_4), U4.5 (A3)
- new net GPIO_AD_B1_10: J4.7 (Pin_7), U4.7 (A5)
- new net GPIO_AD_B1_11: J4.6 (Pin_6), U2.4 (A2)
- new net GPIO_AD_B1_12: J4.19 (Pin_19), U4.4 (A2)
- new net GPIO_AD_B1_13: J4.18 (Pin_18), U4.6 (A4)
- new net GPIO_AD_B1_14: J5.18 (Pin_18), U2.7 (A5)
- new net GPIO_AD_B1_15: J5.19 (Pin_19), U2.6 (A4)
- new net GPIO_B0_00: J5.12 (Pin_12), U4.8 (A6)
- new net GPIO_B0_01: J5.14 (Pin_14), U4.10 (A8)
- new net GPIO_B0_02: J5.13 (Pin_13), U4.9 (A7)
- new net GPIO_B0_03: J4.14 (Pin_14), U2.3 (A1)
- new net GPIO_B0_10: J5.8 (Pin_8), U2.5 (A3)
- new net GPIO_B0_11: J5.11 (Pin_11), U2.8 (A6)
- new net GPIO_B0_12: J5.24 (Pin_24), U6.9 (A7)
- new net GPIO_B1_00: J5.10 (Pin_10), U2.9 (A7)
- new net GPIO_B1_01: J5.9 (Pin_9), U2.10 (A8)
- new net GPIO_B1_02: J4.21 (Pin_21), U3.8 (A6)
- new net GPIO_B1_03: J4.20 (Pin_20), U3.9 (A7)
- new net GPIO_B1_12: J4.22 (Pin_22), U1.10 (A8)
- new net GPIO_B1_13: J4.23 (Pin_23), U5.3 (A1)
- new net GPIO_EMC_04: J5.4 (Pin_4), U3.6 (A4)
- new net GPIO_EMC_05: J5.5 (Pin_5), U3.7 (A5)
- new net GPIO_EMC_06: J5.6 (Pin_6), U3.10 (A8)
- new net GPIO_EMC_07: J4.24 (Pin_24), U5.4 (A2)
- new net GPIO_EMC_08: J5.7 (Pin_7), R7.2, U7.1 (~{INT})
- new net GPIO_EMC_31: J5.21 (Pin_21), J8.6 (Pin_6)
- new net GPIO_EMC_32: J5.20 (Pin_20), U1.6 (A4)
- new net GPIO_EMC_36: J5.23 (Pin_23), U3.5 (A3)
- new net GPIO_EMC_37: J5.22 (Pin_22), U6.10 (A8)
- new net SPARE0: J8.2 (Pin_2), U7.19 (P16)
- new net SPARE1: J8.4 (Pin_4), U7.20 (P17)
- no-connect marks 5 -> 28
Other:
- note added: "3.3V"
- note added: "ON/OFF"
- note added: "PROGRAM"
- moved on the sheet: RN4A, RN4B, RN4C, RN4D
