File: board/pertec_arduino_adapter.kicad_pcb (KiCad board)
At the start: 6 copper layers, 88.9 x 101.6 mm, 48 parts, among them J1 Pertec J1, J2 Pertec J2, J3 Teensy Ethernet, J4 Teensy Right, J5 Teensy Left, J6 Teensy Cross, J7 RJ45_Cetus_J1B1211CCD, Q1 BSS138, Q2 BSS138, U1 SN74LVC8T245NSR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

Commit message: Revision A for tapeout.
Parts:
- JP1: value ISGL/SPCMD1 -> Jumper_3_Open; footprint pertec_arduino_adapter:PinHeader_1x02_P2.54mm_Vertical -> pertec_arduino_adapter:PinHeader_1x03_P2.54mm_Vertical
- RN4: footprint pertec_arduino_adapter:R_Array_SIP6 -> pertec_arduino_adapter:R_Array_SIP10
- moved JP1 3.09 mm to (115.6, 121.5)
- moved RN4 2.54 mm to (149.9, 114.9)
Connections:
- JP1 pad 1: ISGL -> Net-(JP1-Pad1)
- JP1 pad 2: Net-(JP1-Pad2) -> ISGL
- RN4 pad 2: IFBY -> Net-(JP1-Pad1)
- RN4 pad 3: IR2 -> IFBY
- RN4 pad 4: IR3 -> IR2
- RN4 pad 5: unconnected-(RN4-Pad5) -> IR3
- RN4 pad 6: +5V -> unconnected-(RN4-Pad6)
- RN5 pad 7: Net-(JP1-Pad2) -> Net-(JP1-Pad3)
Routing:
- net Net-(JP1-Pad1): track 0.00 -> 39.6 mm
- net +3V3: track 168.5 -> 198.4 mm, vias 4 -> 7
- net ILDP: track 81.6 -> 64.4 mm
- net IFBY: track 75.0 -> 85.5 mm, vias 1 -> 0
- net Net-(JP1-Pad3): track 0.00 -> 4.30 mm
- net Net-(JP1-Pad2): track 4.06 -> 0.00 mm
- net IFAD: track 46.1 -> 42.6 mm
- net IR3: track 37.3 -> 34.1 mm
- net IR2: track 38.2 -> 35.7 mm
- net IWFM: track 57.2 -> 59.6 mm
- net IOFL: track 92.2 -> 90.1 mm
- net ITAD0: track 105.5 -> 107.4 mm
- net ISGL: track 82.6 -> 81.0 mm
- net IRTH1: track 87.9 -> 89.0 mm
- net IDENT: track 53.8 -> 54.9 mm, vias 3 -> 1
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- added copper zone on In2.Cu, net +5V
- added copper zone on In1.Cu, net GNDREF
- removed copper zone on In1.Cu, net +3V3
- removed copper zone on In3.Cu, net +5V
- removed copper zone on In2.Cu, net GNDREF
Other:
- copper layers 6 -> 4
- board text added: "* ISGL a/k/a IDEN0/SPCMD1"
- board text added: "*ISGL"
- board text added: "1"
- board text added: "1-2"
- board text added: "2"
- board text added: "2-3"
- board text added: "3"
- board text added: "Analyzer"
- board text added: "CR2032 3V"
- board text added: "Controller"
- board text added: "Don't care"
- board text added: "Ground"
- board text added: "ICER"
- board text added: "IDBY"
- board text added: "IDEN"
- board text added: "IDENT"
- board text added: "IEDIT"
- board text added: "IEOT"
- board text added: "IERASE"
- board text added: "IFAD"
- board text added: "IFBY"
- board text added: "IFEN"
- board text added: "IFMK"
- board text added: "IFPT"
- board text added: "IGO"
- board text added: "IHER"
- board text added: "ILDP"
- board text added: "ILOL"
- board text added: "ILWD"
- board text added: "INRZ"
- board text added: "IOFL"
- board text added: "IONL"
- board text added: "IR0"
- board text added: "IR1"
- board text added: "IR2"
- board text added: "IR3"
- board text added: "IR4"
- board text added: "IR5"
- board text added: "IR6"
- board text added: "IR7"
- board text added: "IRDY"
- board text added: "IREV"
- board text added: "IREW"
- board text added: "IRP"
- board text added: "IRSTR"
- board text added: "IRTH1"
- board text added: "IRTH2"
- board text added: "IRWD"
- board text added: "ISPEED"
- board text added: "ITAD0"
- board text added: "ITAD1"
- board text added: "IW0"
- board text added: "IW1"
- board text added: "IW2"
- board text added: "IW3"
- board text added: "IW4"
- board text added: "IW5"
- board text added: "IW6"
- board text added: "IW7"
- board text added: "IWFM"
- board text added: "IWP"
- board text added: "IWRT"
- board text added: "IWSTR"
- board text added: "Input (ISGL/IDEN0)"
- board text added: "Input (SPCMD1)"
- board text added: "Input (any)"
- board text added: "Installed"
- board text added: "Italics names are controller inputs/ peripheral outputs."
- board text added: "J1:14"
- board text added: "JP1"
- board text added: "Mode"
- board text added: "Output (ISGL/IDEN0)"
- board text added: "Output (SPCMD1)"
- board text added: "Peripheral"
- board text added: "Pertec J1"
- board text added: "Pertec J2"
- board text added: "Pertexus Pertex adapter for Teensy 4.1 Bjoren Davis bdb004 Revision A May 21, 2022"
- board text added: "RN1-4"
- board text added: "RN5-8"
- board text added: "Uninstalled"
