File: board/pertec_arduino_adapter.kicad_pcb (KiCad board)
At the start: 4 copper layers, 88.9 x 101.6 mm, 48 parts, among them J1 Pertec J1, J2 Pertec J2, J3 Teensy Ethernet, J4 Teensy Right, J5 Teensy Left, J6 Teensy Cross, J7 RJ45_Cetus_J1B1211CCD, Q1 BSS138, Q2 BSS138, U1 SN74LVC8T245NSR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

Commit message: Development checkpoint: revision A1 (added holes for feet)
Parts:
- added REF**: MountingHole_4.3mm_M4_ISO14580, MountingHole:MountingHole_4.3mm_M4_ISO14580, F.Cu at (170.8, 52.7)
- added REF**: MountingHole_4.3mm_M4_ISO14580, MountingHole:MountingHole_4.3mm_M4_ISO14580, F.Cu at (90.2, 119.4)
- added REF**: MountingHole_4.3mm_M4_ISO14580, MountingHole:MountingHole_4.3mm_M4_ISO14580, F.Cu at (170.8, 119.4)
- added REF**: MountingHole_4.3mm_M4_ISO14580, MountingHole:MountingHole_4.3mm_M4_ISO14580, F.Cu at (90.8, 52.7)
- moved RN4 1.27 mm to (149.9, 113.7)
Routing:
- net Net-(JP1-Pad1): track 39.6 -> 40.8 mm
- net IR3: track 34.1 -> 35.2 mm
- net IR2: track 35.7 -> 36.7 mm
- net IFBY: track 85.5 -> 86.5 mm
Other:
- board text added: "Pertexus Pertex adapter for Teensy 4.1 Bjoren Davis bdb004 Revision A1 May 22, 2022"
- board text removed: "Pertexus Pertex adapter for Teensy 4.1 Bjoren Davis bdb004 Revision A May 21, 2022"
