File: board/pertec_arduino_adapter.kicad_sch (KiCad schematic)
At the start: 47 parts, among them J1 Conn_02x25_Odd_Even, J2 Conn_02x25_Odd_Even, J3 Conn_02x03_Odd_Even, J4 Conn_01x24, J5 Conn_01x24, J6 Conn_01x05, Q1 BSS138, Q2 BSS138, U7 PCA9535DBR

Commit message: Development checkpoint: added switchable controller/peripheral functionality.
Parts:
- removed J8: (no value), symbol pertec_arduino_adapter:Conn_02x03_Odd_Even
- removed R10, R11, R9: 10 kΩ, symbol pertec_arduino_adapter:R
- added JP1: ISGL/SPCMD1, symbol pertec_arduino_adapter:Jumper_2_Bridged
- added RN5, RN6, RN7: R1=220Ω, R2=330Ω, pertec_arduino_adapter:R_Array_SIP10, symbol pertec_arduino_adapter:R_DualNetwork_16R
- added RN8: R1=220Ω, R2=330Ω, pertec_arduino_adapter:R_Array_SIP6, symbol pertec_arduino_adapter:R_DualNetwork_8R
- C1: value (none) -> 0.1 μF; footprint (none) -> pertec_arduino_adapter:C_Rect_L4.0mm_W2.5mm_P2.50mm
- C10, C11, C12, C13, C14, C2, C4, C5, C6, C7, C8, C9: footprint (none) -> pertec_arduino_adapter:C_0805_2012Metric_Pad1.18x1.45mm_HandSolder
- C3: value (none) -> 0.1 μF; footprint (none) -> pertec_arduino_adapter:C_0805_2012Metric_Pad1.18x1.45mm_HandSolder
- J7: value (none) -> RJ45_Cetus_J1B1211CCD; footprint (none) -> pertec_arduino_adapter:RJ45_Cetus_J1B1211CCD_Horizontal
- Q1, Q2: footprint (none) -> pertec_arduino_adapter:SOT-23
- R1, R2, R3, R4, R5, R6, R7, R8: footprint (none) -> pertec_arduino_adapter:R_0805_2012Metric_Pad1.20x1.40mm_HandSolder
- U1, U2, U3, U4, U5, U6: value (none) -> SN74LVC8T245NSR; footprint (none) -> pertec_arduino_adapter:SO-24_5.3x15mm_P1.27mm
Connections:
- net SPARE0 is gone; now on net ILDP: U7.19 (P16)
- net SPARE1 is gone; now on net IFPT: U7.20 (P17)
- net +5V: now also RN5.10, RN5.10, RN5.10, RN5.10, RN5.10, RN5.10, RN5.10, RN5.10, RN6.10, RN6.10, RN6.10, RN6.10, RN6.10, RN6.10, RN6.10, RN6.10, RN7.10, RN7.10, RN7.10, RN7.10, RN7.10, RN7.10, RN7.10, RN7.10, RN8.6, RN8.6, RN8.6, RN8.6
- net GNDREF: now also RN5.1, RN5.1, RN5.1, RN5.1, RN5.1, RN5.1, RN5.1, RN5.1, RN6.1, RN6.1, RN6.1, RN6.1, RN6.1, RN6.1, RN6.1, RN6.1, RN7.1, RN7.1, RN7.1, RN7.1, RN7.1, RN7.1, RN7.1, RN7.1, RN8.1, RN8.1, RN8.1, RN8.1; no longer U1.2 (DIR), U1.22 (~{OE}), U3.2 (DIR), U3.22 (~{OE}), U5.2 (DIR), U5.22 (~{OE})
- net IDEN: now also RN7.9
- net IEDIT: now also RN7.3
- net IERASE: now also RN7.4
- net IFAD: now also RN8.5
- net IFEN: now also RN8.2
- net IFPT: no longer U3.17 (B5)
- net IGO: now also RN5.4
- net ILDP: no longer U1.18 (B4)
- net ILOL: now also RN5.8
- net ILWD: now also RN5.2
- net IOFL: now also RN8.3
- net IREV: now also RN5.9
- net IREW: now also RN6.2
- net IRTH1: now also RN7.6
- net IRTH2: now also RN7.2
- net ISGL: now also JP1.1 (A)
- net ITAD0: now also RN7.7
- net ITAD1: now also RN8.4
- net IW0: now also RN5.5
- net IW1: now also RN5.6
- net IW2: now also RN6.7
- net IW3: now also RN6.5
- net IW4: now also RN5.3
- net IW5: now also RN6.8
- net IW6: now also RN6.6
- net IW7: now also RN6.4
- net IWFM: now also RN7.5
- net IWP: now also RN6.3
- net IWRT: now also RN6.9
- net DIRB: now reaches U4.2 (DIR)
- net DIRB: now also J5.20 (Pin_20), U2.2 (DIR), U6.2 (DIR)
- net GPIO_AD_B0_02 renamed LVIRP
- net GPIO_AD_B0_03 renamed LVIFMK
- net GPIO_AD_B0_12 renamed LPI2C4_SCL
- net GPIO_AD_B0_13 renamed LPI2C4_SDA
- net GPIO_AD_B1_00 renamed LVIR7
- net GPIO_AD_B1_01 renamed LVIR6
- net GPIO_AD_B1_02 renamed LVIR5
- net GPIO_AD_B1_03 renamed LVIR4
- net GPIO_AD_B1_04 renamed LVIR3
- net GPIO_AD_B1_05 renamed LVIR2
- net GPIO_AD_B1_06 renamed LVIR1
- net GPIO_AD_B1_07 renamed LVIR0
- net GPIO_AD_B1_08 renamed LVIW7
- net GPIO_AD_B1_09 renamed LVIW6
- net GPIO_AD_B1_10 renamed LVIW5
- net GPIO_AD_B1_11 renamed LVIW4
- net GPIO_AD_B1_12 renamed LVIW3
- net GPIO_AD_B1_13 renamed LVIW2
- net GPIO_AD_B1_14 renamed LVIW1
- net GPIO_AD_B1_15 renamed LVIW0
- net GPIO_B0_00 renamed LVIWRT
- net GPIO_B0_01 renamed LVIERASE
- net GPIO_B0_02 renamed LVIEDIT
- net GPIO_B0_03 renamed LVILWD
- net GPIO_B0_10 renamed LVIGO
- net GPIO_B0_11 renamed LVIREV
- net GPIO_B0_12 renamed LVIWFM
- net GPIO_B1_00 renamed LVIREW
- net GPIO_B1_01 renamed LVIWP
- net GPIO_B1_02 renamed LVIRSTR
- net GPIO_B1_03 renamed LVIWSTR
- net GPIO_B1_12 renamed LVIHER
- net GPIO_B1_13 renamed LVICER
- net GPIO_EMC_04 renamed LVIRDY
- net GPIO_EMC_05: no longer names the net of U3.7 (A5)
- net GPIO_EMC_05: no longer J5.5 (Pin_5)
- net GPIO_EMC_06 renamed LVIDBY
- net GPIO_EMC_07 renamed LVIFBY
- net GPIO_EMC_08 renamed ~{LPI2C4_INT}
- net GPIO_EMC_31 renamed OEA
- net OEA: now also U1.22 (~{OE}), U3.22 (~{OE}), U5.22 (~{OE})
- net GPIO_EMC_32: no longer names the net of U1.6 (A4)
- net GPIO_EMC_32: no longer J5.20 (Pin_20)
- net GPIO_EMC_36 renamed LVIEOT
- net GPIO_EMC_37 renamed LVIOFL
- new net: JP1.2 (B), RN5.7
- new net DIRA: J5.5 (Pin_5), U1.2 (DIR), U3.2 (DIR), U5.2 (DIR)
- no-connect marks 28 -> 33
Other:
- note added: "A (Bold)"
- note added: "B (Unbolded)"
- note added: "Controller"
- note added: "GPIO_AD_B0_02"
- note added: "GPIO_AD_B0_03"
- note added: "GPIO_AD_B0_12"
- note added: "GPIO_AD_B0_13"
- note added: "GPIO_AD_B1_00"
- note added: "GPIO_AD_B1_01"
- note added: "GPIO_AD_B1_02"
- note added: "GPIO_AD_B1_03"
- note added: "GPIO_AD_B1_04"
- note added: "GPIO_AD_B1_05"
- note added: "GPIO_AD_B1_06"
- note added: "GPIO_AD_B1_07"
- note added: "GPIO_AD_B1_08"
- note added: "GPIO_AD_B1_09"
- note added: "GPIO_AD_B1_10"
- note added: "GPIO_AD_B1_11"
- note added: "GPIO_AD_B1_12"
- note added: "GPIO_AD_B1_13"
- note added: "GPIO_AD_B1_14"
- note added: "GPIO_AD_B1_15"
- note added: "GPIO_B0_00"
- note added: "GPIO_B0_01"
- note added: "GPIO_B0_02"
- note added: "GPIO_B0_03"
- note added: "GPIO_B0_10"
- note added: "GPIO_B0_11"
- note added: "GPIO_B0_12"
- note added: "GPIO_B1_00"
- note added: "GPIO_B1_01"
- note added: "GPIO_B1_02"
- note added: "GPIO_B1_03"
- note added: "GPIO_B1_12"
- note added: "GPIO_B1_13"
- note added: "GPIO_EMC_04"
- note added: "GPIO_EMC_05"
- note added: "GPIO_EMC_06"
- note added: "GPIO_EMC_07"
- note added: "GPIO_EMC_08"
- note added: "GPIO_EMC_31"
- note added: "GPIO_EMC_32"
- note added: "GPIO_EMC_36"
- note added: "GPIO_EMC_37"
- note added: "Group A: Termination for controller inputs."
- note added: "Group B: Termination for peripheral inputs."
- note added: "Input"
- note added: "Mode"
- note added: "Output"
- note added: "Peripheral"
- note added: "Signal Group"
- moved on the sheet: BT1, C10, C11, C12, C13, C14, C2, C3, C4, C5, C6, C7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

Commit message: Development checkpoint: ready to start layout
Parts:
- renumbered U3 to U2, U5 to U3, U6 to U5, U2 to U6
Other:
- moved on the sheet: J4, J5, U1, U2, U3, U4, U5, U6

Commit message: Development checkpoint: fully routed.  Still 6 layers, but I'll chop that down right before tapeout.
Parts:
- removed RN8: R1=220Ω, R2=330Ω, pertec_arduino_adapter:R_Array_SIP6, symbol pertec_arduino_adapter:R_DualNetwork_8R
- added RN8: R1=220Ω, R2=330Ω, pertec_arduino_adapter:R_Array_SIP10, symbol pertec_arduino_adapter:R_DualNetwork_16R
- JP1: footprint (none) -> pertec_arduino_adapter:PinHeader_1x02_P2.54mm_Vertical
Connections:
- net +3V3: now also J6.4 (Pin_4)
- net +5V: now also RN8.10, RN8.10, RN8.10, RN8.10, RN8.10, RN8.10, RN8.10, RN8.10
- net GNDREF: now also RN8.1, RN8.1, RN8.1, RN8.1, RN8.1, RN8.1, RN8.1, RN8.1
- net IDEN: now also RN8.6; no longer RN7.9
- net IFAD: now also RN8.5
- net IFEN: now also RN8.2
- net IOFL: now also RN8.3
- net ITAD1: now also RN8.4
- no-connect marks 33 -> 36

Commit message: Development checkpoint: layout and routing completed; passes DRC
Parts:
- J1, J2: value Conn_02x25_Odd_Even -> (none)
- J3: value Conn_02x03_Odd_Even -> (none); footprint pertec_arduino_adapter:PinSocket_2x03_P2.00mm_Vertical_Mirror -> (none)
- J4, J5: value Conn_01x24 -> (none); footprint pertec_arduino_adapter:PinSocket_1x24_P2.54mm_Vertical -> (none)
- J6: value Conn_01x05 -> (none); footprint pertec_arduino_adapter:PinSocket_1x05_P2.54mm_Vertical -> (none)

Commit message: Revision A for tapeout.
Parts:
- removed JP1: ISGL/SPCMD1, pertec_arduino_adapter:PinHeader_1x02_P2.54mm_Vertical, symbol pertec_arduino_adapter:Jumper_2_Bridged
- removed RN4: R1=220Ω, R2=330Ω, pertec_arduino_adapter:R_Array_SIP6, symbol pertec_arduino_adapter:R_DualNetwork_8R
- added JP1: Jumper_3_Open, pertec_arduino_adapter:PinHeader_1x03_P2.54mm_Vertical, symbol pertec_arduino_adapter:Jumper_3_Open
- added RN4: R1=220Ω, R2=330Ω, pertec_arduino_adapter:R_Array_SIP10, symbol pertec_arduino_adapter:R_DualNetwork_16R
- J1: value (none) -> Pertec J1
- J2: value (none) -> Pertec J2
- J3: value (none) -> Teensy Ethernet; footprint (none) -> pertec_arduino_adapter:PinSocket_2x03_P2.00mm_Vertical_Mirror_Teensy4.1_J3
- J4: value (none) -> Teensy Right; footprint (none) -> pertec_arduino_adapter:PinSocket_1x24_P2.54mm_Vertical_Teensy4.1_J4
- J5: value (none) -> Teensy Left; footprint (none) -> pertec_arduino_adapter:PinSocket_1x24_P2.54mm_Vertical_Teensy4.1_J5
- J6: value (none) -> Teensy Cross; footprint (none) -> pertec_arduino_adapter:PinSocket_1x05_P2.54mm_Vertical_Teensy4.1_J6
Connections:
- net +5V: now also RN4.10, RN4.10, RN4.10, RN4.10, RN4.10, RN4.10, RN4.10, RN4.10
- net GNDREF: now also RN4.1, RN4.1, RN4.1, RN4.1, RN4.1, RN4.1, RN4.1, RN4.1
- net IFBY: now also RN4.3
- net IR2: now also RN4.4
- net IR3: now also RN4.5
- net ISGL: now also JP1.2 (C)
- net at RN5.7: now also JP1.3 (B)
- new net: JP1.1 (A), RN4.2
- no-connect marks 36 -> 39
Other:
- title: Pertec Arduino Adapter (bdb004) -> Pertexus: A Teensy 4.1 (Arduino) Pertex Interface (bdb004)
- moved on the sheet: RN1A, RN1B, RN1C, RN1D, RN1E, RN1F, RN1G, RN1H, RN2A, RN2B, RN2C, RN2D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
